File: ROBOTCircuitBoard.kicad_pcb (KiCad board)
At the start: 2 copper layers, 0 parts

Commit message: finished the component libraries
Parts:
- added C10: 2.2uF, Capacitors_SMD:C_0805, F.Cu at (161.3, 94.0)
- added C11: 2.2uF, Capacitors_SMD:C_0805, F.Cu at (166.4, 94.0)
- added C12: CP 0.1uF, Capacitors_SMD:C_0603, F.Cu at (125.7, 108.0)
- added C2: 2.2uF, Capacitors_SMD:C_0805, F.Cu at (161.3, 88.9)
- added C3: CP 0.1uF, Capacitors_SMD:C_0603, F.Cu at (123.2, 95.2)
- added C4: 0.1uF, Capacitors_SMD:C_0603, F.Cu at (175.3, 97.8)
- added C5: 2.2uF, Capacitors_SMD:C_0805, F.Cu at (142.2, 105.4)
- added C6: 0.1uF, Capacitors_SMD:C_0603, F.Cu at (143.5, 101.6)
- added C7: CP 0.1uF, Capacitors_SMD:C_0603, F.Cu at (175.3, 102.9)
- added C8: 0.1uF, Capacitors_SMD:C_0603, F.Cu at (175.3, 106.7)
- added C9: CP 2.2uF, Capacitors_SMD:C_0805, F.Cu at (171.4, 94.0)
- added D1: LED, LEDs:LED_1206, F.Cu at (144.8, 67.3)
- added D2: D_Schottky_AAK, Diodes_SMD:D_SOT-23_ANK, F.Cu at (158.8, 110.5)
- added F1: Fuse, Fuse_Holders_and_Fuses:Fuse_SMD1206_Reflow, F.Cu at (147.3, 115.6)
- added J3: CONN_01X02, Pin_Headers:Pin_Header_Straight_1x02_Pitch2.54mm, F.Cu at (115.6, 101.6)
- added L1: L Ferrite, Capacitors_SMD:C_0603, F.Cu at (130.8, 118.1)
- added L2: L Ferrite, Capacitors_SMD:C_0603, F.Cu at (133.3, 116.8)
- added P3: Pushbutton NO, Buttons_Switches_SMD:SW_SPST_PTS810, F.Cu at (111.8, 113.0)
- added P4: USB_OTG, Connectors:USB_Micro-B, F.Cu at (151.1, 87.6)
- added R1: 470, Resistors_SMD:R_0201, F.Cu at (152.4, 71.1)
- added R2: 470, Resistors_SMD:R_0201, F.Cu at (170.2, 102.9)
- added R3: 33, Resistors_SMD:R_0201, F.Cu at (148.6, 110.5)
- added R4: 33, Resistors_SMD:R_0201, F.Cu at (154.9, 101.6)
- added U2: MK20DX256VLH7, MK20DX256VLH7:QFP50P1200X1200X160-64N, F.Cu at (133.3, 86.4)
- added U3: LP38691, kicadfootprints:lp38691, F.Cu at (109.2, 87.6)
- added U4: MKL02, Teensy_DIY_v1.0:Teensy_DIY_v1.0-QFN50P300X300X100-17N, F.Cu at (133.3, 99.1)
- added Y1: Crystal 16MHz, Crystals:Crystal_AT310_d3.0mm_l10.0mm_Horizontal, F.Cu at (134.6, 66.0)
