File: ROBOTCircuitBoard.sch (KiCad schematic (older format))
At the start: 27 parts, among them J3 CONN_01X02, P3 Pushbutton NO, P4 USB_OTG, U2 MK20DX256VLH7, U3 LP38691, U4 MKL02, Y1 Crystal 16MHz

Commit message: made a lp38691 footprint
Parts:
- U3: footprint (none) -> kicadfootprints:lp38691
Changed lines of the file:
@@
 F 0 "U3" H 4750 2900 60  0000 C CNN
 F 1 "LP38691" H 4750 3300 60  0000 C CNN
-F 2 "" H 4750 3100 60  0001 C CNN
+F 2 "kicadfootprints:lp38691" H 4750 3100 60  0001 C CNN
 F 3 "" H 4750 3100 60  0001 C CNN
 	1    4750 3100

Commit message: added libraries
Parts:
- U2: footprint QFP50P1200X1200X160-64N -> MK20DX256VLH7:QFP50P1200X1200X160-64N
Changed lines of the file:
@@
 F 0 "U2" H 2410 7630 50  0000 L CNN
 F 1 "MK20DX256VLH7" H 2350 3300 50  0000 L CNN
-F 2 "QFP50P1200X1200X160-64N" H 2550 5400 50  0001 L CNN
+F 2 "MK20DX256VLH7:QFP50P1200X1200X160-64N" H 2550 5400 50  0001 L CNN
 F 3 "Freescale Semiconductor" H 2550 5400 50  0001 L CNN
 F 4 "MCU 32-bit Kinetis K20 ARM Cortex M4 RISC 256KB Flash 1.8V/2.5V/3.3V 64-Pin LQFP Tray" H 2550 5400 50  0001 L CNN "Description"

Commit message: finished the component libraries
Parts:
- U4: footprint (none) -> Teensy_DIY_v1.0:Teensy_DIY_v1.0-QFN50P300X300X100-17N
- Y1: footprint (none) -> Crystals:Crystal_AT310_d3.0mm_l10.0mm_Horizontal
Changed lines of the file:
@@
 F 0 "U4" H 5250 5400 60  0000 C CNN
 F 1 "MKL02" H 5250 6500 60  0000 C CNN
-F 2 "" H 5250 6000 60  0001 C CNN
+F 2 "Teensy_DIY_v1.0:Teensy_DIY_v1.0-QFN50P300X300X100-17N" H 5250 6000 60  0001 C CNN
 F 3 "" H 5250 6000 60  0001 C CNN
 	1    5250 6000
@@
 F 0 "Y1" H 1100 6650 50  0000 C CNN
 F 1 "Crystal 16MHz" H 1100 6350 50  0000 C CNN
-F 2 "" H 1100 6500 50  0001 C CNN
+F 2 "Crystals:Crystal_AT310_d3.0mm_l10.0mm_Horizontal" H 1100 6500 50  0001 C CNN
 F 3 "" H 1100 6500 50  0000 C CNN
 	1    1100 6500

Commit message: updated netlist, soread out objects
Parts:
- added J1: Analog 9-0, Socket_Strips:Socket_Strip_Straight_1x10_Pitch1.27mm, symbol CONN_01X10
Connections:
- wire segments 67 -> 68
Other:
- moved on the sheet: D1, R1
Changed lines of the file:
@@
 L LED D1
 U 1 1 598FA689
-P 1200 4850
-F 0 "D1" H 1200 4950 50  0000 C CNN
-F 1 "LED" H 1200 4750 50  0000 C CNN
-F 2 "LEDs:LED_1206" H 1200 4850 50  0001 C CNN
-F 3 "" H 1200 4850 50  0001 C CNN
-	1    1200 4850
+P 1000 4850
+F 0 "D1" H 1000 4950 50  0000 C CNN
+F 1 "LED" H 1000 4750 50  0000 C CNN
+F 2 "LEDs:LED_1206" H 1000 4850 50  0001 C CNN
+F 3 "" H 1000 4850 50  0001 C CNN
+	1    1000 4850
 	1    0    0    -1
 $EndComp
@@
 L R R1
 U 1 1 598FA746
-P 900 4850
-F 0 "R1" V 980 4850 50  0000 C CNN
-F 1 "470" V 900 4850 50  0000 C CNN
-F 2 "Resistors_SMD:R_0201" V 830 4850 50  0001 C CNN
-F 3 "" H 900 4850 50  0001 C CNN
-	1    900  4850
+P 700 4850
+F 0 "R1" V 780 4850 50  0000 C CNN
+F 1 "470" V 700 4850 50  0000 C CNN
+F 2 "Resistors_SMD:R_0201" V 630 4850 50  0001 C CNN
+F 3 "" H 700 4850 50  0001 C CNN
+	1    700  4850
 	0    1    1    0
 $EndComp
@@
 L GND #PWR011
 U 1 1 598FA803
-P 750 4850
-F 0 "#PWR011" H 750 4600 50  0001 C CNN
-F 1 "GND" H 750 4700 50  0000 C CNN
-F 2 "" H 750 4850 50  0001 C CNN
-F 3 "" H 750 4850 50  0001 C CNN
-	1    750  4850
+P 550 4850
+F 0 "#PWR011" H 550 4600 50  0001 C CNN
+F 1 "GND" H 550 4700 50  0000 C CNN
+F 2 "" H 550 4850 50  0001 C CNN
+F 3 "" H 550 4850 50  0001 C CNN
+	1    550  4850
 	1    0    0    -1
 $EndComp
@@
 Wire Wire Line
 	4000 2950 4000 2900
+$Comp
+L CONN_01X10 J1
+U 1 1 59CEF135
+P 1150 5400
+F 0 "J1" H 1150 5950 50  0000 C CNN
+F 1 "Analog 9-0" V 1250 5400 50  0000 C CNN
+F 2 "Socket_Strips:Socket_Strip_Straight_1x10_Pitch1.27mm" H 1150 5400 50  0001 C CNN
+F 3 "" H 1150 5400 50  0001 C CNN
+	1    1150 5400
+	-1   0    0    1
+$EndComp
+Wire Wire Line
+	1150 4850 1350 4850
 $EndSCHEMATC
